File: DAC Outputs_0_10V.kicad_sch (KiCad schematic)
At the start: 30 parts, among them J12 1862411, J13 1862411, J14 1862411, J15 1862411, J16 1862411, J17 1862411, J18 1862411, J19 1862411, U7 DAC8568ICPW, U8 OPA4192IDR, U9 OPA4192IDR

Commit message: Updated schematic and PCB
Parts:
- removed C36: 100nF, Capacitor_SMD:C_0805_2012Metric, symbol Device:C
- removed J12, J13, J14, J15, J16, J17, J18, J19: 1862411, CONN_1862411, symbol PC Term Block 2 Pos 45deg:1862411
- removed U9: OPA4192IDR, D0014A_N, symbol 2026-03-28_20-43-41:OPA4192IDR
- added J7: 1190365, LPTA 2,5 4-5,0:PHOENIX_1190365, symbol 1190365:1190365
- added J8: 1190374, LPTA 2,512-5,0 - PCB terminal block1:PHOENIX_1190374, symbol 1190374:1190374
- added U13, U14, U17, U9: XTR111AxDGQ, Package_SO:MSOP-10-1EP_3x3mm_P0.5mm_EP2.2x3.1mm_Mask1.83x1.89mm_ThermalVias, symbol Interface_CurrentLoop:XTR111AxDGQ
- R37, R38, R41, R42: value 10k -> 100
- R39, R40, R43, R44: value 10k -> 20k
Connections:
- net +24V: now also U13.1 (VSP), U14.1 (VSP), U17.1 (VSP), U9.1 (VSP)
- net AO4: now also U9.6 (VIN)
- net AO5: now also U13.6 (VIN)
- net AO6: now also U14.6 (VIN)
- net AO7: now also U17.6 (VIN)
- net GND: now also R37.1, R38.1, R39.2, R41.1, R42.1, R43.2, J7.2_1, J7.2_2, J7.4_1, J7.4_2, J8.10_1, J8.10_2, J8.12_1, J8.12_2, J8.2_1, J8.2_2, J8.4_1, J8.4_2, J8.6_1, J8.6_2, J8.8_1, J8.8_2, U13.10 (GND), U13.11 (GND), U13.5 (REGF), U14.10 (GND), U14.11 (GND), U14.5 (REGF), U17.10 (GND), U17.11 (GND), U17.5 (REGF), U9.10 (GND), U9.11 (GND), U9.5 (REGF); no longer R38.2, R42.2
- net A0: now reaches R29.1, U8.1 (OUT)
- net A0: now also J7.1_1, J7.1_2
- net at R37.2: now also U9.3 (VG), U9.4 (REGS); no longer R38.1
- net at R41.2: now also U14.3 (VG), U14.4 (REGS); no longer R42.1
- net at R43.1: now also U14.7 (SET)
- net at R44.1: now also U17.7 (SET); no longer R43.2
- net at R40.1: now also U13.7 (SET); no longer R39.2
- net A3: now reaches R35.1, U8.14 (OUT)
- net A3: now also J8.3_1, J8.3_2
- net A2: now reaches R33.1, U8.8 (OUT)
- net A2: now also J8.1_1, J8.1_2
- net at R39.1: now also U9.7 (SET)
- net A1: now reaches R31.1, U8.7 (OUT)
- net A1: now also J7.3_1, J7.3_2
- new net: R38.2, U13.3 (VG), U13.4 (REGS)
- new net: R42.2, U17.3 (VG), U17.4 (REGS)
- new net A4: J8.5_1, J8.5_2, U9.2 (IS)
- new net A5: J8.7_1, J8.7_2, U13.2 (IS)
- new net A6: J8.9_1, J8.9_2, U14.2 (IS)
- new net A7: J8.11_1, J8.11_2, U17.2 (IS)
Other:
- moved on the sheet: R31, R32, R35, R36, U8B, U8D
