File: DAC_Outputs_4_20mA .kicad_sch (KiCad schematic)
At the start: 18 parts, among them J24 1862411, J25 1862411, J26 1862411, J27 1862411, U10 DAC8568ICPW, U11 XTR111AxDGQ, U12 XTR111AxDGQ, U13 XTR111AxDGQ, U14 XTR111AxDGQ

Commit message: Updated schematic and PCB
Parts:
- removed C37: 2.2uF, Capacitor_SMD:C_0805_2012Metric, symbol Device:C
- removed J24, J25, J26, J27: 1862411, CONN_1862411, symbol PC Term Block 2 Pos 45deg:1862411
- removed R45, R47, R51, R52: 100, Resistor_SMD:R_0805_2012Metric, symbol Device:R
- removed R46, R48, R49, R53: 20k, Resistor_SMD:R_0805_2012Metric, symbol Device:R
- removed U10: DAC8568ICPW, DAC8568ICPW:SOP65P640X120-16N, symbol DAC8568ICPW:DAC8568ICPW
- removed U11, U12, U13, U14: XTR111AxDGQ, Package_SO:MSOP-10-1EP_3x3mm_P0.5mm_EP2.2x3.1mm_Mask1.83x1.89mm_ThermalVias, symbol Interface_CurrentLoop:XTR111AxDGQ
